File: tart_radio_module/tart_radio_module.kicad_sch (KiCad schematic)
At the start: 34 parts, among them J2 RFShield_OnePiece, J3 Conn_Coaxial, J4 Conn_Coaxial, U3 MAX2769B

Commit message: update
Parts:
- U3: footprint Package_DFN_QFN:TQFN-28-1EP_5x5mm_P0.5mm_EP3.25x3.25mm_ThermalVias -> tart_radio_module:MAX2769B
Changed lines of the file:
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@@
 			)
 		)
-		(property "Footprint" "Package_DFN_QFN:TQFN-28-1EP_5x5mm_P0.5mm_EP3.25x3.25mm_ThermalVias"
+		(property "Footprint" "tart_radio_module:MAX2769B"
 			(at 140.716 139.446 0)
 			(effects
@@
 		)
 	)
+	(sheet_instances
+		(path "/"
+			(page "1")
+		)
+	)
