File: tart_radio_module/tart_radio_module.kicad_pcb (KiCad board)
At the start: 6 copper layers, 35.5 x 15 mm, 34 parts, among them J1 Conn_Coaxial, J2 RFShield_OnePiece, J3 Conn_Coaxial, U1 MAX2769B

Commit message: update
Parts:
- U1: footprint Package_DFN_QFN:TQFN-28-1EP_5x5mm_P0.5mm_EP3.25x3.25mm_ThermalVias -> tart_radio_module:MAX2769B
Other:
- board text added: "CLKOUT"
Changed lines of the file:
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@@
 		)
 	)
-	(footprint "Package_DFN_QFN:TQFN-28-1EP_5x5mm_P0.5mm_EP3.25x3.25mm_ThermalVias"
+	(footprint "tart_radio_module:MAX2769B"
 		(locked yes)
 		(layer "F.Cu")
 		(at 125 103 90)
-		(descr "TQFN, 28 Pin (https://pdfserv.maximintegrated.com/package_dwgs/21-0140.PDF (T2855-3)), generated with kicad-footprint-generator ipc_noLead_generator.py")
-		(tags "TQFN NoLead")
+		(descr "MAX2769B (https://www.analog.com/en/products/max2769b.html)")
 		(property "Reference" "U1"
 			(at 0 -3.8 90)
@@
 			(at 0 3.8 90)
 			(layer "F.Fab")
-			(hide yes)
 			(effects
 				(font
@@
 			)
 		)
-		(property "Footprint" "Package_DFN_QFN:TQFN-28-1EP_5x5mm_P0.5mm_EP3.25x3.25mm_ThermalVias"
+		(property "Footprint" "tart_radio_module:MAX2769B"
 			(at 0 0 90)
 			(layer "F.Fab")
@@
 			(pintype "power_in")
 		)
-		(model "${KICAD8_3DMODEL_DIR}/Package_DFN_QFN.3dshapes/TQFN-28-1EP_5x5mm_P0.5mm_EP3.25x3.25mm.wrl"
+		(model "${KIPRJMOD}/tart_radio_module.pretty/MAX2769B.stp"
 			(offset
 				(xyz 0 0 0)
@@
 		(layer "Edge.Cuts")
 	)
+	(gr_text "CLKOUT"
+		(at 136.25 98 0)
+		(layer "F.SilkS")
+		(effects
+			(font
+				(size 0.5 0.5)
+				(thickness 0.1)
+				(bold yes)
+			)
+		)
+	)
 	(gr_text "PWR"
