File: tart_frontend.kicad_pcb (KiCad board)
At the start: 6 copper layers, 45.8 x 62 mm, 146 parts, among them J10 Conn_Coaxial, J11 RFShield_OnePiece, J12 Conn_Coaxial, J13 Conn_Coaxial, J2 RFShield_OnePiece, J3 Conn_Coaxial, J4 Conn_Coaxial, J5 RFShield_OnePiece, J6 Conn_Coaxial, J7 Conn_Coaxial, J8 RFShield_OnePiece, J9 Conn_Coaxial, U1 CDCV304PW, U2 MAX3280E, U3 MAX2769B, U4 MAX2769B, U5 MAX2769B, U6 MAX2769B

Commit message: update
Parts:
- removed C10, C14, C17, C18, C26, C30, C33, C34, C42, C46, C49, C50, C58, C62, C65, C66: 100nF, Capacitor_SMD:C_0402_1005Metric
- removed C11, C13, C21, C23, C24, C27, C29, C37, C39, C40, C43, C45, C5, C53, C55, C56, C59, C61, C7, C8: 10nF, Capacitor_SMD:C_0402_1005Metric
- removed C12, C28, C44, C60: 100pF, Capacitor_SMD:C_0402_1005Metric
- removed C15, C31, C47, C63: 47nF, Capacitor_SMD:C_0402_1005Metric
- removed C16, C32, C48, C64: 27pF, Capacitor_SMD:C_0402_1005Metric
- removed C19, C20, C3, C35, C36, C4, C51, C52: 10uF, Capacitor_SMD:C_0603_1608Metric
- removed C22, C25, C38, C41, C54, C57, C6, C9: 0.47nF, Capacitor_SMD:C_0402_1005Metric
- removed D1, D10, D11, D12, D2, D3, D4, D5, D6, D7, D8, D9: LED, Diode_SMD:D_0603_1608Metric
- removed FB1, FB2, FB3, FB4: GZ1608D601TF, Inductor_SMD:L_0603_1608Metric
- removed J10, J13, J4, J7: Conn_Coaxial, tart_radio_module:CONN-SMD_MOLEX_73412-0110
- removed J11, J2, J5, J8: RFShield_OnePiece, RF_Shielding:Laird_Technologies_BMI-S-101_13.66x12.70mm
- removed J12, J3, J6, J9: Conn_Coaxial, tart_radio_module:CONN-SMD_KH-SMA-KE8-G
- removed L1, L2, L3, L4: L, Inductor_SMD:L_0402_1005Metric
- removed R10, R11, R17, R18, R19, R20, R26, R27, R28, R29, R35, R36, R37, R38, R8, R9: 100, Resistor_SMD:R_0402_1005Metric
- removed R12, R15, R16, R21, R24, R25, R30, R33, R34, R39, R6, R7: 1k, Resistor_SMD:R_0402_1005Metric
- removed R13, R22, R31, R4: 1k, Resistor_SMD:R_0603_1608Metric
- removed R14, R23, R32, R5: 20k, Resistor_SMD:R_0402_1005Metric
- removed U3, U4, U5, U6: MAX2769B, Package_DFN_QFN:TQFN-28-1EP_5x5mm_P0.5mm_EP3.25x3.25mm_ThermalVias

Commit message: update
Parts:
- added C10: 100nF, Capacitor_SMD:C_0402_1005Metric, F.Cu at (31.8, 59.9)
- added C11: 10nF, Capacitor_SMD:C_0402_1005Metric, F.Cu at (31.8, 61.9)
- added C12: 100pF, Capacitor_SMD:C_0402_1005Metric, F.Cu at (31.8, 63.9)
- added C13: 10nF, Capacitor_SMD:C_0402_1005Metric, F.Cu at (31.8, 65.8)
- added C14: 100nF, Capacitor_SMD:C_0402_1005Metric, F.Cu at (31.8, 67.8)
- added C15: 47nF, Capacitor_SMD:C_0402_1005Metric, F.Cu at (34.7, 59.9)
- added C16: 27pF, Capacitor_SMD:C_0402_1005Metric, F.Cu at (34.7, 61.9)
- added C17: 100nF, Capacitor_SMD:C_0402_1005Metric, F.Cu at (34.7, 63.9)
- added C18: 100nF, Capacitor_SMD:C_0402_1005Metric, F.Cu at (34.7, 65.8)
- added C19: 10uF, Capacitor_SMD:C_0603_1608Metric, F.Cu at (46.8, 91.5)
- added C20: 10uF, Capacitor_SMD:C_0603_1608Metric, F.Cu at (46.8, 94.0)
- added C21: 10nF, Capacitor_SMD:C_0402_1005Metric, F.Cu at (28.9, 91.2)
- added C22: 0.47nF, Capacitor_SMD:C_0402_1005Metric, F.Cu at (28.9, 93.2)
- added C23: 10nF, Capacitor_SMD:C_0402_1005Metric, F.Cu at (28.9, 95.2)
- added C24: 10nF, Capacitor_SMD:C_0402_1005Metric, F.Cu at (28.9, 97.1)
- added C25: 0.47nF, Capacitor_SMD:C_0402_1005Metric, F.Cu at (28.9, 99.1)
- added C26: 100nF, Capacitor_SMD:C_0402_1005Metric, F.Cu at (31.8, 91.2)
- added C27: 10nF, Capacitor_SMD:C_0402_1005Metric, F.Cu at (31.8, 93.2)
- added C28: 100pF, Capacitor_SMD:C_0402_1005Metric, F.Cu at (31.8, 95.2)
- added C29: 10nF, Capacitor_SMD:C_0402_1005Metric, F.Cu at (31.8, 97.1)
- added C3: 10uF, Capacitor_SMD:C_0603_1608Metric, F.Cu at (46.8, 60.2)
- added C30: 100nF, Capacitor_SMD:C_0402_1005Metric, F.Cu at (31.8, 99.1)
- added C31: 47nF, Capacitor_SMD:C_0402_1005Metric, F.Cu at (34.7, 91.2)
- added C32: 27pF, Capacitor_SMD:C_0402_1005Metric, F.Cu at (34.7, 93.2)
- added C33: 100nF, Capacitor_SMD:C_0402_1005Metric, F.Cu at (34.7, 95.2)
- added C34: 100nF, Capacitor_SMD:C_0402_1005Metric, F.Cu at (34.7, 97.1)
- added C35: 10uF, Capacitor_SMD:C_0603_1608Metric, F.Cu at (75.7, 91.5)
- added C36: 10uF, Capacitor_SMD:C_0603_1608Metric, F.Cu at (75.7, 94.0)
- added C37: 10nF, Capacitor_SMD:C_0402_1005Metric, F.Cu at (57.8, 91.2)
- added C38: 0.47nF, Capacitor_SMD:C_0402_1005Metric, F.Cu at (57.8, 93.2)
- added C39: 10nF, Capacitor_SMD:C_0402_1005Metric, F.Cu at (57.8, 95.2)
- added C4: 10uF, Capacitor_SMD:C_0603_1608Metric, F.Cu at (46.8, 62.7)
- added C40: 10nF, Capacitor_SMD:C_0402_1005Metric, F.Cu at (57.8, 97.1)
- added C41: 0.47nF, Capacitor_SMD:C_0402_1005Metric, F.Cu at (57.8, 99.1)
- added C42: 100nF, Capacitor_SMD:C_0402_1005Metric, F.Cu at (60.7, 91.2)
- added C43: 10nF, Capacitor_SMD:C_0402_1005Metric, F.Cu at (60.7, 93.2)
- added C44: 100pF, Capacitor_SMD:C_0402_1005Metric, F.Cu at (60.7, 95.2)
- added C45: 10nF, Capacitor_SMD:C_0402_1005Metric, F.Cu at (60.7, 97.1)
- added C46: 100nF, Capacitor_SMD:C_0402_1005Metric, F.Cu at (60.7, 99.1)
- added C47: 47nF, Capacitor_SMD:C_0402_1005Metric, F.Cu at (63.6, 91.2)
- added C48: 27pF, Capacitor_SMD:C_0402_1005Metric, F.Cu at (63.6, 93.2)
- added C49: 100nF, Capacitor_SMD:C_0402_1005Metric, F.Cu at (63.6, 95.2)
- added C5: 10nF, Capacitor_SMD:C_0402_1005Metric, F.Cu at (28.9, 59.9)
- added C50: 100nF, Capacitor_SMD:C_0402_1005Metric, F.Cu at (63.6, 97.1)
- added C51: 10uF, Capacitor_SMD:C_0603_1608Metric, F.Cu at (75.7, 60.2)
- added C52: 10uF, Capacitor_SMD:C_0603_1608Metric, F.Cu at (75.7, 62.7)
- added C53: 10nF, Capacitor_SMD:C_0402_1005Metric, F.Cu at (57.8, 59.9)
- added C54: 0.47nF, Capacitor_SMD:C_0402_1005Metric, F.Cu at (57.8, 61.9)
- added C55: 10nF, Capacitor_SMD:C_0402_1005Metric, F.Cu at (57.8, 63.9)
- added C56: 10nF, Capacitor_SMD:C_0402_1005Metric, F.Cu at (57.8, 65.8)
- added C57: 0.47nF, Capacitor_SMD:C_0402_1005Metric, F.Cu at (57.8, 67.8)
- added C58: 100nF, Capacitor_SMD:C_0402_1005Metric, F.Cu at (60.7, 59.9)
- added C59: 10nF, Capacitor_SMD:C_0402_1005Metric, F.Cu at (60.7, 61.9)
- added C6: 0.47nF, Capacitor_SMD:C_0402_1005Metric, F.Cu at (28.9, 61.9)
- added C60: 100pF, Capacitor_SMD:C_0402_1005Metric, F.Cu at (60.7, 63.9)
- added C61: 10nF, Capacitor_SMD:C_0402_1005Metric, F.Cu at (60.7, 65.8)
- added C62: 100nF, Capacitor_SMD:C_0402_1005Metric, F.Cu at (60.7, 67.8)
- added C63: 47nF, Capacitor_SMD:C_0402_1005Metric, F.Cu at (63.6, 59.9)
- added C64: 27pF, Capacitor_SMD:C_0402_1005Metric, F.Cu at (63.6, 61.9)
- added C65: 100nF, Capacitor_SMD:C_0402_1005Metric, F.Cu at (63.6, 63.9)
- added C66: 100nF, Capacitor_SMD:C_0402_1005Metric, F.Cu at (63.6, 65.8)
- added C7: 10nF, Capacitor_SMD:C_0402_1005Metric, F.Cu at (28.9, 63.9)
- added C8: 10nF, Capacitor_SMD:C_0402_1005Metric, F.Cu at (28.9, 65.8)
- added C9: 0.47nF, Capacitor_SMD:C_0402_1005Metric, F.Cu at (28.9, 67.8)
- added D1: LED, Diode_SMD:D_0603_1608Metric, F.Cu at (52.3, 44.2)
- added D10: LED, Diode_SMD:D_0603_1608Metric, F.Cu at (81.2, 44.2)
- added D11: LED, Diode_SMD:D_0603_1608Metric, F.Cu at (81.2, 46.8)
- added D12: LED, Diode_SMD:D_0603_1608Metric, F.Cu at (81.2, 49.4)
- added D2: LED, Diode_SMD:D_0603_1608Metric, F.Cu at (52.3, 46.8)
- added D3: LED, Diode_SMD:D_0603_1608Metric, F.Cu at (52.3, 49.4)
- added D4: LED, Diode_SMD:D_0603_1608Metric, F.Cu at (52.3, 75.5)
- added D5: LED, Diode_SMD:D_0603_1608Metric, F.Cu at (52.3, 78.1)
- added D6: LED, Diode_SMD:D_0603_1608Metric, F.Cu at (52.3, 80.7)
- added D7: LED, Diode_SMD:D_0603_1608Metric, F.Cu at (81.2, 75.5)
- added D8: LED, Diode_SMD:D_0603_1608Metric, F.Cu at (81.2, 78.1)
- added D9: LED, Diode_SMD:D_0603_1608Metric, F.Cu at (81.2, 80.7)
- added FB1: GZ1608D601TF, Inductor_SMD:L_0603_1608Metric, F.Cu at (46.8, 65.2)
- added FB2: GZ1608D601TF, Inductor_SMD:L_0603_1608Metric, F.Cu at (46.8, 96.5)
- added FB3: GZ1608D601TF, Inductor_SMD:L_0603_1608Metric, F.Cu at (75.7, 96.5)
- added FB4: GZ1608D601TF, Inductor_SMD:L_0603_1608Metric, F.Cu at (75.7, 65.2)
- added J10: Conn_Coaxial, tart_radio_module:CONN-SMD_MOLEX_73412-0110, F.Cu at (80.5, 93.0)
- added J11: RFShield_OnePiece, RF_Shielding:Laird_Technologies_BMI-S-101_13.66x12.70mm, F.Cu at (63.9, 50.9)
- added J12: Conn_Coaxial, tart_radio_module:CONN-SMD_KH-SMA-KE8-G, F.Cu at (75.3, 55.7)
- added J13: Conn_Coaxial, tart_radio_module:CONN-SMD_MOLEX_73412-0110, F.Cu at (80.5, 61.7)
- added J2: RFShield_OnePiece, RF_Shielding:Laird_Technologies_BMI-S-101_13.66x12.70mm, F.Cu at (35.0, 50.9)
- added J3: Conn_Coaxial, tart_radio_module:CONN-SMD_KH-SMA-KE8-G, F.Cu at (46.4, 55.7)
- added J4: Conn_Coaxial, tart_radio_module:CONN-SMD_MOLEX_73412-0110, F.Cu at (51.6, 61.7)
- added J5: RFShield_OnePiece, RF_Shielding:Laird_Technologies_BMI-S-101_13.66x12.70mm, F.Cu at (35.0, 82.2)
- added J6: Conn_Coaxial, tart_radio_module:CONN-SMD_KH-SMA-KE8-G, F.Cu at (46.4, 86.9)
- added J7: Conn_Coaxial, tart_radio_module:CONN-SMD_MOLEX_73412-0110, F.Cu at (51.6, 93.0)
- added J8: RFShield_OnePiece, RF_Shielding:Laird_Technologies_BMI-S-101_13.66x12.70mm, F.Cu at (63.9, 82.2)
- added J9: Conn_Coaxial, tart_radio_module:CONN-SMD_KH-SMA-KE8-G, F.Cu at (75.3, 86.9)
- added L1: L, Inductor_SMD:L_0402_1005Metric, F.Cu at (37.6, 60.0)
- added L2: L, Inductor_SMD:L_0402_1005Metric, F.Cu at (37.6, 91.2)
- added L3: L, Inductor_SMD:L_0402_1005Metric, F.Cu at (66.5, 91.2)
- added L4: L, Inductor_SMD:L_0402_1005Metric, F.Cu at (66.5, 60.0)
- added R10: 100, Resistor_SMD:R_0402_1005Metric, F.Cu at (43.4, 60.0)
- added R11: 100, Resistor_SMD:R_0402_1005Metric, F.Cu at (43.4, 61.9)
- added R12: 1k, Resistor_SMD:R_0402_1005Metric, F.Cu at (43.4, 63.9)
- added R13: 1k, Resistor_SMD:R_0603_1608Metric, F.Cu at (46.8, 99.0)
- added R14: 20k, Resistor_SMD:R_0402_1005Metric, F.Cu at (37.6, 93.2)
- added R15: 1k, Resistor_SMD:R_0402_1005Metric, F.Cu at (37.6, 95.2)
- added R16: 1k, Resistor_SMD:R_0402_1005Metric, F.Cu at (40.5, 91.2)
- added R17: 100, Resistor_SMD:R_0402_1005Metric, F.Cu at (40.5, 93.2)
- added R18: 100, Resistor_SMD:R_0402_1005Metric, F.Cu at (40.5, 95.2)
- added R19: 100, Resistor_SMD:R_0402_1005Metric, F.Cu at (43.4, 91.2)
- added R20: 100, Resistor_SMD:R_0402_1005Metric, F.Cu at (43.4, 93.2)
- added R21: 1k, Resistor_SMD:R_0402_1005Metric, F.Cu at (43.4, 95.2)
- added R22: 1k, Resistor_SMD:R_0603_1608Metric, F.Cu at (75.7, 99.0)
- added R23: 20k, Resistor_SMD:R_0402_1005Metric, F.Cu at (66.5, 93.2)
- added R24: 1k, Resistor_SMD:R_0402_1005Metric, F.Cu at (66.5, 95.2)
- added R25: 1k, Resistor_SMD:R_0402_1005Metric, F.Cu at (69.4, 91.2)
- added R26: 100, Resistor_SMD:R_0402_1005Metric, F.Cu at (69.4, 93.2)
- added R27: 100, Resistor_SMD:R_0402_1005Metric, F.Cu at (69.4, 95.2)
- added R28: 100, Resistor_SMD:R_0402_1005Metric, F.Cu at (72.3, 91.2)
- added R29: 100, Resistor_SMD:R_0402_1005Metric, F.Cu at (72.3, 93.2)
- added R30: 1k, Resistor_SMD:R_0402_1005Metric, F.Cu at (72.3, 95.2)
- added R31: 1k, Resistor_SMD:R_0603_1608Metric, F.Cu at (75.7, 67.7)
- added R32: 20k, Resistor_SMD:R_0402_1005Metric, F.Cu at (66.5, 61.9)
- added R33: 1k, Resistor_SMD:R_0402_1005Metric, F.Cu at (66.5, 63.9)
- added R34: 1k, Resistor_SMD:R_0402_1005Metric, F.Cu at (69.4, 60.0)
- added R35: 100, Resistor_SMD:R_0402_1005Metric, F.Cu at (69.4, 61.9)
- added R36: 100, Resistor_SMD:R_0402_1005Metric, F.Cu at (69.4, 63.9)
- added R37: 100, Resistor_SMD:R_0402_1005Metric, F.Cu at (72.3, 60.0)
- added R38: 100, Resistor_SMD:R_0402_1005Metric, F.Cu at (72.3, 61.9)
- added R39: 1k, Resistor_SMD:R_0402_1005Metric, F.Cu at (72.3, 63.9)
- added R4: 1k, Resistor_SMD:R_0603_1608Metric, F.Cu at (46.8, 67.7)
- added R5: 20k, Resistor_SMD:R_0402_1005Metric, F.Cu at (37.6, 61.9)
- added R6: 1k, Resistor_SMD:R_0402_1005Metric, F.Cu at (37.6, 63.9)
- added R7: 1k, Resistor_SMD:R_0402_1005Metric, F.Cu at (40.5, 60.0)
- added R8: 100, Resistor_SMD:R_0402_1005Metric, F.Cu at (40.5, 61.9)
- added R9: 100, Resistor_SMD:R_0402_1005Metric, F.Cu at (40.5, 63.9)
- added U3: MAX2769B, tart_radio_module:MAX2769B, F.Cu at (39.7, 68.5)
- added U4: MAX2769B, tart_radio_module:MAX2769B, F.Cu at (39.7, 99.8)
- added U5: MAX2769B, tart_radio_module:MAX2769B, F.Cu at (68.6, 99.8)
- added U6: MAX2769B, tart_radio_module:MAX2769B, F.Cu at (68.6, 68.5)

Commit message: update
Parts:
- removed C10, C14, C17, C18, C26, C30, C33, C34, C42, C46, C49, C50, C58, C62, C65, C66: 100nF, Capacitor_SMD:C_0402_1005Metric
- removed C11, C13, C21, C23, C24, C27, C29, C37, C39, C40, C43, C45, C5, C53, C55, C56, C59, C61, C7, C8: 10nF, Capacitor_SMD:C_0402_1005Metric
- removed C12, C28, C44, C60: 100pF, Capacitor_SMD:C_0402_1005Metric
- removed C15, C31, C47, C63: 47nF, Capacitor_SMD:C_0402_1005Metric
- removed C16, C32, C48, C64: 27pF, Capacitor_SMD:C_0402_1005Metric
- removed C19, C20, C3, C35, C36, C4, C51, C52: 10uF, Capacitor_SMD:C_0603_1608Metric
- removed C22, C25, C38, C41, C54, C57, C6, C9: 0.47nF, Capacitor_SMD:C_0402_1005Metric
- removed D1, D10, D11, D12, D2, D3, D4, D5, D6, D7, D8, D9: LED, Diode_SMD:D_0603_1608Metric
- removed FB1, FB2, FB3, FB4: GZ1608D601TF, Inductor_SMD:L_0603_1608Metric
- removed J10, J13, J4, J7: Conn_Coaxial, tart_radio_module:CONN-SMD_MOLEX_73412-0110
- removed J11, J2, J5, J8: RFShield_OnePiece, RF_Shielding:Laird_Technologies_BMI-S-101_13.66x12.70mm
- removed J12, J3, J6, J9: Conn_Coaxial, tart_radio_module:CONN-SMD_KH-SMA-KE8-G
- removed L1, L2, L3, L4: L, Inductor_SMD:L_0402_1005Metric
- removed R10, R11, R17, R18, R19, R20, R26, R27, R28, R29, R35, R36, R37, R38, R8, R9: 100, Resistor_SMD:R_0402_1005Metric
- removed R12, R15, R16, R21, R24, R25, R30, R33, R34, R39, R6, R7: 1k, Resistor_SMD:R_0402_1005Metric
- removed R13, R22, R31, R4: 1k, Resistor_SMD:R_0603_1608Metric
- removed R14, R23, R32, R5: 20k, Resistor_SMD:R_0402_1005Metric
- removed U3, U4, U5, U6: MAX2769B, tart_radio_module:MAX2769B
